File: schematics/2025_power/2025_power.kicad_pcb (KiCad board)
At the start: 2 copper layers, 70.5 x 66.8 mm, 30 parts, among them J1 Conn_01x02, J10 Conn_01x02, J2 Conn_01x02, J3 Conn_01x02, J4 Conn_01x02, J5 Conn_01x02, J6 Conn_01x02, J7 Conn_01x02, J8 Conn_01x02, J9 Conn_01x02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

Commit message: 2025 power revised
Parts:
- added C10: 10u, Capacitor_SMD:CP_Elec_4x5.4, F.Cu at (96.5, 92.3)
- added C5: 100u, Capacitor_SMD:CP_Elec_6.3x7.7, F.Cu at (114.7, 99.0)
- added C6: 220u, Capacitor_SMD:CP_Elec_6.3x7.7, F.Cu at (99.7, 68.3)
- added C7: 100u, Capacitor_SMD:CP_Elec_6.3x7.7, F.Cu at (108.5, 63.3)
- added C8: 22u, Capacitor_SMD:CP_Elec_6.3x5.4, F.Cu at (94.0, 85.8)
- C4: value 470u -> 220u; footprint Capacitor_SMD:CP_Elec_10x10 -> Capacitor_SMD:CP_Elec_6.3x7.7
- H1, H2, TP1: moved to B.Cu
- J1, J2: footprint Connector_JST:JST_XH_S2B-XH-A_1x02_P2.50mm_Horizontal -> Connector_JST:JST_VH_B2PS-VH_1x02_P3.96mm_Horizontal
- J10, J3, J4, J5, J6, J7, J8, J9: footprint Connector_JST:JST_XH_S2B-XH-A_1x02_P2.50mm_Horizontal -> Connector_JST:JST_XH_B2B-XH-A_1x02_P2.50mm_Vertical
- R1: value 10k -> 22k
- R4: value 1k -> 22k
- RV1: value 10k -> 20k; footprint PCM_SL_Devices:potentiometer_3362P -> Potentiometer_SMD:Potentiometer_Bourns_3314J_Vertical
- SW1: value SW_SPDT -> VS14-0123ZWZ03-6; footprint my_footprint:SW_SPDT_2.5mm -> kicad-gemini-generated:Legion VS14-0123ZWZ03-6
- moved H1 60.7 mm to (139.7, 115.4), turned to 180 degrees
- moved J9 59.4 mm to (79.1, 78.9), turned to -62 degrees
- moved J4 50.7 mm to (83.3, 86.7), turned to -62 degrees
- moved C1 50.4 mm to (137.5, 103.8)
- moved J10 41.7 mm to (87.6, 94.4), turned to -62 degrees
- moved J6 41.7 mm to (130.6, 84.8), turned to 120 degrees
- moved SW1 35.8 mm to (125.7, 108.2)
- moved TP5 34.7 mm to (119.0, 74.4), turned to 120 degrees
- moved C4 33.6 mm to (135.2, 93.0), turned to 180 degrees
- moved J5 32.8 mm to (91.8, 102.4), turned to -62 degrees
- moved J3 32.4 mm to (126.0, 76.7), turned to 120 degrees
- moved C2 31.5 mm to (89.7, 76.0), turned to -150 degrees
- moved D3 31.4 mm to (120.4, 85.9), turned to 30 degrees
- moved TP2 29.7 mm to (116.0, 88.9), turned to 120 degrees
- moved L1 28.4 mm to (114.4, 79.4), turned to 120 degrees
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Connections:
- C4 pad 1: V+ -> +V_SW
- J1 pad 1: GND -> +12V
- J1 pad 2: +12V -> GND
- J10 pad 1: GND -> V+
- J10 pad 2: V+ -> GND
- J2 pad 1: GND -> +12V
- J2 pad 2: +12V -> GND
- J3 pad 1: GND -> V+
- J3 pad 2: V+ -> GND
- J4 pad 1: GND -> V+
- J4 pad 2: V+ -> GND
- J5 pad 1: GND -> V+
- J5 pad 2: V+ -> GND
- J6 pad 1: GND -> V+
- J6 pad 2: V+ -> GND
- J7 pad 1: GND -> V+
- J7 pad 2: V+ -> GND
- J8 pad 1: GND -> V+
- J8 pad 2: V+ -> GND
- J9 pad 1: GND -> V+
- J9 pad 2: V+ -> GND
- SW1 pad 1: +V_SW -> +12V
- SW1 pad 2: +12V -> +V_SW
Routing:
- net GND: track 4.13 -> 11.0 mm, vias 22 -> 83
- net Net-(D3-K): track 2.74 -> 0.00 mm
- net Vsense: track 22.7 -> 24.9 mm, vias 3 -> 4
- net +V_SW: track 0.00 -> 1.91 mm
- net V+: vias 111 -> 0
- removed copper zone on B.Cu, net V+
Other:
- outline, holes or cut-outs redrawn
- board text added: "+"
- board text added: "GND"
- board text added: "In"
- board text added: "L"
- board text added: "ON"
- board text added: "S"
- board text added: "Vout"
