File: schematics/2025_power/2025_power.kicad_sch (KiCad schematic)
At the start: 30 parts, among them J1 Conn_01x02, J10 Conn_01x02, J2 Conn_01x02, J3 Conn_01x02, J4 Conn_01x02, J5 Conn_01x02, J6 Conn_01x02, J7 Conn_01x02, J8 Conn_01x02, J9 Conn_01x02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

Commit message: 2025 power revised
Parts:
- removed SW1: SW_SPDT, my_footprint:SW_SPDT_2.5mm, symbol Switch:SW_SPDT
- added C10: 10u, Capacitor_SMD:CP_Elec_4x5.4, symbol Device:C_Polarized
- added C5, C7: 100u, Capacitor_SMD:CP_Elec_6.3x7.7, symbol Device:C_Polarized
- added C6: 220u, Capacitor_SMD:CP_Elec_6.3x7.7, symbol Device:C_Polarized
- added C8: 22u, Capacitor_SMD:CP_Elec_6.3x5.4, symbol Device:C_Polarized
- added SW1: VS14-0123ZWZ03-6, kicad-gemini-generated:Legion VS14-0123ZWZ03-6, symbol mylib:SW_Legion_VS14-0123ZWZ03-6
- C4: value 470u -> 220u; footprint Capacitor_SMD:CP_Elec_10x10 -> Capacitor_SMD:CP_Elec_6.3x7.7; LCSC C3350 -> C2918361
- J1, J2: footprint Connector_JST:JST_XH_S2B-XH-A_1x02_P2.50mm_Horizontal -> Connector_JST:JST_VH_B2PS-VH_1x02_P3.96mm_Horizontal; LCSC C157931 -> C158007
- J10, J3, J4, J5, J6, J7, J8, J9: footprint Connector_JST:JST_XH_S2B-XH-A_1x02_P2.50mm_Horizontal -> Connector_JST:JST_XH_B2B-XH-A_1x02_P2.50mm_Vertical; LCSC C157931 -> C158012
- R1: value 10k -> 22k; LCSC C25744 -> C25547
- RV1: value 10k -> 20k; footprint PCM_SL_Devices:potentiometer_3362P -> Potentiometer_SMD:Potentiometer_Bourns_3314J_Vertical; LCSC C58159 -> C55069
Connections:
- net +12V: now also J1.1 (Pin_1), J2.1 (Pin_1), SW1.1, SW1.5; no longer J1.2 (Pin_2), J2.2 (Pin_2)
- net +V_SW: now also C4.1, C5.1, SW1.2, SW1.6
- net GND: now also J1.2 (Pin_2), J2.2 (Pin_2), C10.2, C5.2, C6.2, C7.2, C8.2; no longer J1.1 (Pin_1), J2.1 (Pin_1)
- net V+: now also C10.1, C6.1, C7.1, C8.1; no longer C4.1
- no-connect marks 3 -> 6
Other:
- moved on the sheet: C2, J1, J2, TP2
